File: AxxSolder.kicad_sch (KiCad schematic)
At the start: 95 parts, among them IC1 LTC4440AHMS8E-5#PBF, IC2 STM32G431KBT6, IC3 TMP236AQDBZRQ1, IC4 OPA2333AIDRBR, IC5 STM32G431KBT6, IC6 TPS54302DDCR, J1 Conn_01x07_Male, J4 Conn_01x07_Male, Q2 2N7002NXAKR, U1 PEC11L-4220F-S0015, U2 BSC014N04LS

Commit message: import USB-PD hardware from AxxSolder
Parts:
- removed F1: 10A Fuse, 3557-2:3557-2, symbol Device:Fuse
- removed IC3: TMP236AQDBZRQ1, TMP236AQDBZRQ1:SOT95P237X112-3N, symbol TMP236AQDBZRQ1:TMP236AQDBZRQ1
- removed J4: Conn_01x07_Male, Connector_PinSocket_2.54mm:PinSocket_1x07_P2.54mm_Vertical, symbol Connector:Conn_01x07_Male
- removed TP1: AmbTemp_TP, TestPoint:TestPoint_THTPad_D1.0mm_Drill0.5mm, symbol Connector:TestPoint
- removed TP2: TestPoint, TestPoint:TestPoint_Pad_D1.0mm, symbol Connector:TestPoint
- added C30: 1u, Capacitor_SMD:C_0805_2012Metric, symbol Device:C_Small
- added C31: 100n, Capacitor_SMD:C_0805_2012Metric, symbol Device:C_Small
- added D10: ESDA25W, ESDA25W:SOT65P210X110-3N, symbol ESDA25W:ESDA25W
- added D11: 1N5819HW-7-F, 1N5819HW-7-F:SOD3716X145N, symbol 1N5819HW-7-F:1N5819HW-7-F
- added D13: V7NM103-M3_I, V7NM103-M3_I:V7NM103M3I, symbol V7NM103-M3_I:V7NM103-M3_I
- added D8: ESDA25P35-1U1M, ESDA25P35-1U1M:ESDA25P351U1M, symbol ESDA25P35-1U1M:ESDA25P35-1U1M
- added F2: 0154007.DRL, 0154007:0154100DR, symbol 0154007_DRL:0154007.DRL
- added IC7: STUSB4500QTR, STUSB4500QTR:QFN50P400X400X100-25N-D, symbol STUSB4500QTR:STUSB4500QTR
- added IC8: USBLC6-2P6, USBLC6-2P6:USBLC62P6, symbol USBLC6-2P6:USBLC6-2P6
- added J2: USB_B_Micro, USB3140-30-0230-1-C_REVE1:GCT_USB3140-30-0230-1-C_REVE1, symbol Connector:USB_B_Micro
- added J5: USB4105-GF-A-120, USB4105-GF-A:GCT_USB4105-GF-A-120, symbol USB4105-GF-A-120:USB4105-GF-A-120
- added J6: Conn_01x06_Socket, Connector_PinSocket_2.54mm:PinSocket_1x06_P2.54mm_Vertical, symbol Connector:Conn_01x06_Socket
- added JP1, JP2: SolderJumper_2_Open, Jumper:SolderJumper-2_P1.3mm_Open_TrianglePad1.0x1.5mm, symbol Jumper:SolderJumper_2_Open
- added Q1: STL9P3LLH6, STL9P3LLH6:STL20N6F7, symbol STL9P3LLH6:STL9P3LLH6
- added R27, R30: 4k7, Resistor_SMD:R_0805_2012Metric, symbol Device:R_Small
- added R31, R35: 1k, Resistor_SMD:R_0805_2012Metric, symbol Device:R_Small
- added R32, R34: 22k, Resistor_SMD:R_0805_2012Metric, symbol Device:R_Small
- added R33: 100k, Resistor_SMD:R_0805_2012Metric, symbol Device:R_Small
- added S2: KMR211G_LFS, KMR211G_LFS:KMR_2, symbol KMR211G_LFS:KMR211G_LFS
- C1, C12, C14, C19, C6: Manufacturer_Name (none) -> Murata Electronics; Manufacturer_Part_Number (none) -> GRM21BR6YA106ME43L
- C10, C11, C13, C2, C21, C22, C24, C28, C29, C3, C7, C8, C9: Manufacturer_Name (none) -> Murata Electronics; Manufacturer_Part_Number (none) -> GRM21BR72A104KAC4L
- C15, C16: Manufacturer_Name (none) -> Murata Electronics; Manufacturer_Part_Number (none) -> GRM2165C1H102JA01D
- C17, C18: Manufacturer_Name (none) -> TDK; Manufacturer_Part_Number (none) -> C3216X5R1V226M160AC
- C20: value 100n -> 1u; Manufacturer_Name (none) -> Murata Electronics; Manufacturer_Part_Number (none) -> GRM21BC72A105KE01L
- C25, C27: Manufacturer_Name (none) -> TDK; Manufacturer_Part_Number (none) -> C2012X6S1C226M125AC
- C26: Manufacturer_Name (none) -> Murata Electronics; Manufacturer_Part_Number (none) -> GRM21A5C2E750FW01D
- C4: value 22u/16V -> 22u; Manufacturer_Name (none) -> TDK; Manufacturer_Part_Number (none) -> C2012X6S1C226M125AC
- C5: value 100n -> 10u; Manufacturer_Name (none) -> Murata Electronics; Manufacturer_Part_Number (none) -> GRM21BR6YA106ME43L
- D1, D12, D3, D5, D6: Manufacturer_Name (none) -> Diotec Semiconductor; Manufacturer_Part_Number (none) -> BAT54S
- D4: Assembly Comment (none) -> Do not Purchase nor assemble; Manufacturer_Name (none) -> N/A; Manufacturer_Part_Number (none) -> N/A
- D9: footprint DIOM5436X261N -> SMBJ24CA:DIOM5436X261N
- H1, H2, H3, H4, TP3, TP5, TP6, TP7, TP8, TP9: Assembly Comment (none) -> N/A; now left out of the parts list
- J1: Manufacturer_Name (none) -> Wurth Elektronik
- PS1: footprint SOT230P700X190-4N -> LD1117AS33TR:SOT230P700X190-4N
- R1, R17, R25, R26, R5, R6: Manufacturer_Name (none) -> Panasonic; Manufacturer_Part_Number (none) -> ERJ-6ENF4701V
- R10: Manufacturer_Name (none) -> Vishay / Dale; Manufacturer_Part_Number (none) -> WSLP25122L500FEA
- R11, R12, R13, R14, R16, R18, R8, R9: Manufacturer_Name (none) -> Panasonic; Manufacturer_Part_Number (none) -> ERJ-6ENF1002V
- R15: Manufacturer_Name (none) -> Panasonic; Manufacturer_Part_Number (none) -> ERJ-6ENF2200V
- R19, R20: Manufacturer_Name (none) -> Panasonic; Manufacturer_Part_Number (none) -> ERJ-6ENF1501V
- R2: Manufacturer_Name (none) -> Panasonic; Manufacturer_Part_Number (none) -> ERJ-6ENF4702V
- R21, R22: Manufacturer_Name (none) -> Panasonic; Manufacturer_Part_Number (none) -> ERJ-6ENF4703V
- R23, R24: Manufacturer_Name (none) -> Panasonic; Manufacturer_Part_Number (none) -> ERJ-6ENF2203V
- R28: Manufacturer_Name (none) -> Panasonic; Manufacturer_Part_Number (none) -> ERJ-6ENF1003V
- R29: Manufacturer_Name (none) -> Panasonic; Manufacturer_Part_Number (none) -> ERJ-6ENF1332V
- R3: Manufacturer_Name (none) -> Panasonic; Manufacturer_Part_Number (none) -> ERJ-6ENF6801V
- R4, R7, TC1, TC2: Assembly Comment (none) -> N/A
- U2: Manufacturer_Name (none) -> Infineon Technologies; Manufacturer_Part_Number (none) -> BSC014N04LSATMA1
Connections:
- net +3.3V: now also J6.2 (Pin_2), R27.2, R30.2, S2.1; no longer C5.1
- net +5V: now also D11.1
- net Buzzer: now also IC2.31 (PB8-BOOT0), IC5.31 (PB8-BOOT0), R14.2, S2.2; no longer IC2.10 (PA5), IC5.10 (PA5)
- net ENC_Button: now also IC2.29 (PB6), IC5.29 (PB6); no longer IC2.19 (PA9), IC5.19 (PA9)
- net GND: now also C5.1, D4.6 (CS), C30.2, D10.3 (ANODE), D8.2 (A), IC7.10 (GND), IC7.12 (ADDR0), IC7.13 (ADDR1), IC7.22 (VSYS), IC7.25 (EP), IC7.6 (RESET), IC8.2 (GND), J2.5 (GND), J2.6 (Shield), J5.A1_B12 (GND), J5.B1_A12 (GND), J5.S1 (SHELL_GND), J5.S2 (SHELL_GND), J5.S3 (SHELL_GND), J5.S4 (SHELL_GND), J6.1 (Pin_1); no longer C5.2
- net Handle_inp: now also C28.1, IC2.19 (PA9), IC5.19 (PA9); no longer IC2.20 (PA10), IC5.20 (PA10)
- net Handle_sense: no longer C28.1
- net MCU_TX: now also J6.6 (Pin_6)
- net NRST: now also J6.3 (Pin_3)
- net SPI_DC: now also IC2.2 (PF0-OSC_IN), IC5.2 (PF0-OSC_IN); no longer IC2.22 (PA12), IC5.22 (PA12)
- net SWCLK: now also J6.4 (Pin_4)
- net SWDIO: now also J6.5 (Pin_5)
- net Stand_inp: now also C29.1, IC2.20 (PA10), IC5.20 (PA10); no longer IC2.21 (PA11), IC5.21 (PA11)
- net Stand_sense: no longer C29.1
- net VDD: now also C31.2, F2.1, R35.2
- net VDD_IN: now reaches D9.2, J1.7 (Pin_7)
- net VDD_IN: now also D13.1 (K), F2.2
- net HEATER_2: now reaches IC2.18 (PA8), IC5.18 (PA8)
- net Identification_inp: now reaches IC2.3 (PF1-OSC_OUT), IC5.3 (PF1-OSC_OUT)
- net SDA: now reaches IC2.30 (PB7), IC5.30 (PB7)
- net SDA: now also IC7.8 (SDA), R30.1
- net Ambient_temp renamed Heater_1
- net Heater_1: now also IC1.1 (INP), R18.1; no longer C20.1
- net Current renamed Current_1
- net Heater renamed Current_2
- net Current_2: no longer IC1.1 (INP), R18.1
- net MCU_RX renamed SCL
- net SCL: now also IC7.7 (SCL), R27.1
- removed net SPI_CS: D4.6 (CS), IC2.29 (PB6), IC5.29 (PB6)
- net Thermocouple renamed Thermocouple_1
- new net: C30.1, IC7.21 (VREG_1V2)
- new net: J5.A7 (DN1), J5.B7 (DN2), JP2.2 (B)
- new net: D10.1 (CATHODE_1), IC7.4 (CC2), IC7.5 (CC2DB), J5.B5 (CC2)
- new net: D10.2 (CATHODE_2), IC7.1 (CC1DB), IC7.2 (CC1), J5.A5 (CC1)
- new net: J5.A6 (DP1), J5.B6 (DP2), JP1.2 (B)
- new net: D13.2 (A), Q1.5 (D)
- new net: C31.1, R34.2
- new net: IC7.16 (VBUS_EN_SNK), R32.1
- new net: IC7.9 (DISCH), R35.1
- new net: C20.1, IC7.23 (VREG_2V7)
- new net: IC7.18 (VBUS_VS_DISCH), R31.1
- new net Thermocouple_2: IC2.10 (PA5), IC5.10 (PA5)
- new net USB_D+: IC2.22 (PA12), IC5.22 (PA12), IC8.6 (I/O1_2)
- new net USB_D-: IC2.21 (PA11), IC5.21 (PA11), IC8.4 (I/O2_2)
- new net USB_DN: IC8.3 (I/O2_1), J2.2 (D-), JP2.1 (A)
- new net USB_DP: IC8.1 (I/O1_1), J2.3 (D+), JP1.1 (A)
- new net USB_PD_GATE: Q1.4 (G), R32.2, R33.1, R34.1
- new net VBUS: C5.2, D8.1 (K), IC7.24 (VDD), J5.A4_B9 (VBUS), J5.B4_A9 (VBUS), Q1.1 (S_1), Q1.2 (S_2), Q1.3 (S_3), R31.2, R33.2
- new net V_BUS: D11.2, IC8.5 (VBUS), J2.1 (VBUS)
Other:
- note added: "7A Fuse"
- note added: "AxxSolder V3.0 JBC Soldering Iron Controller"
- note added: "Firmware update USB"
- note removed: "AxxSolder V2.2 JBC Soldering Iron Controller"
- note removed: "TEMPERATURE SENSOR"
- moved on the sheet: C28, C29, C8, D9, R12, R14
